File: Hardware/Explorador.sch (KiCad schematic (older format))
At the start: 18 parts, among them CON1 JACK CARGA, Q1 BD244, U1 LM317T, U2 LM2940 - 5.0V

Commit message: Añadidos Sensores
Parts:
- added U?: SHT15, symbol SHT15
- added U?: Ultrasonidos_PING, symbol Ultrasonidos_PING
- BT1: value 7,2v/2000mA -> 7,2v/2600mA
Connections:
- net GND: now also U?.1 (GND), U?.4 (GND)
- net VCC: now also U?.1 (VCC), U?.2 (VCC)
Changed lines of the file:
@@
 LIBS:contrib
 LIBS:valves
-LIBS:freetronics_schematic
-LIBS:arduino
 LIBS:relays
 LIBS:battery_management
 LIBS:Power_Management
 LIBS:elec-unifil
+LIBS:Mi_Libreria_Arduino
+LIBS:arduino
 LIBS:Explorador-cache
 EELAYER 25 0
@@
 P 1350 1750
 F 0 "BT1" H 1100 1800 50  0000 L CNN
-F 1 "7,2v/2000mA" H 800 1700 50  0000 L CNN
+F 1 "7,2v/2600mA" H 800 1700 50  0000 L CNN
 F 2 "Connectors_Molex:Molex_KK-6410-02_02x2.54mm_Straight" V 1350 1810 50  0001 C CNN
 F 3 "" V 1350 1810 50  0000 C CNN
@@
 F 0 "U1" H 4150 2250 50  0000 C CNN
 F 1 "LM317T" H 4700 2250 50  0000 L CNN
-F 2 "Power_Integrations:TO-220" H 4350 2150 50  0000 C CIN
+F 2 "Power_Integrations:TO-220" H 4350 2150 50  0001 C CIN
 F 3 "" H 4350 2050 50  0000 C CNN
 	1    4350 2050
@@
 F 0 "U2" H 5000 804 50  0000 C CNN
 F 1 "LM2940 - 5.0V" H 4850 1200 50  0000 C CNN
-F 2 "Power_Integrations:TO-220" H 4850 1000 50  0000 C CNN
+F 2 "Power_Integrations:TO-220" H 4850 1000 50  0001 C CNN
 F 3 "" H 4850 1000 50  0000 C CNN
 	1    4850 1000
@@
 	4850 1250 4850 1550
 Wire Wire Line
-	4450 1400 4450 1550
-Wire Wire Line
 	3950 950  4450 950
 Connection ~ 4450 950
@@
 Wire Wire Line
 	3150 1800 3150 2600
+Wire Wire Line
+	4450 1400 4450 1550
+$Comp
+L SHT15 U?
+U 1 1 58AB69DA
+P 8700 950
+F 0 "U?" H 8700 950 60  0000 C BNN
+F 1 "SHT15" H 8750 450 60  0000 C TNN
+F 2 "" H 8700 950 60  0001 C CNN
+F 3 "" H 8700 950 60  0001 C CNN
+	1    8700 950
+	1    0    0    -1
+$EndComp
+$Comp
+L VCC #PWR?
+U 1 1 58AB6B1C
+P 9050 800
+F 0 "#PWR?" H 9050 650 50  0001 C CNN
+F 1 "VCC" H 9050 950 50  0000 C CNN
+F 2 "" H 9050 800 50  0000 C CNN
+F 3 "" H 9050 800 50  0000 C CNN
+	1    9050 800
+	1    0    0    -1
+$EndComp
+Wire Wire Line
+	9050 1050 9050 800
+Wire Wire Line
+	9050 1050 8850 1050
+$Comp
+L GND #PWR?
+U 1 1 58AB7157
+P 9050 1600
+F 0 "#PWR?" H 9050 1350 50  0001 C CNN
+F 1 "GND" H 9050 1450 50  0001 C CNN
+F 2 "" H 9050 1600 50  0000 C CNN
+F 3 "" H 9050 1600 50  0000 C CNN
+	1    9050 1600
+	1    0    0    -1
+$EndComp
+Wire Wire Line
+	8850 1350 9050 1350
+Wire Wire Line
+	9050 1350 9050 1600
+$Comp
+L Ultrasonidos_PING U?
+U 1 1 58AB72A4
+P 9900 1000
+F 0 "U?" H 9900 1050 60  0000 C CNN
+F 1 "Ultrasonidos_PING" H 9900 1150 60  0000 C CNN
+F 2 "" H 9900 1000 60  0001 C CNN
+F 3 "" H 9900 1000 60  0001 C CNN
+	1    9900 1000
+	1    0    0    -1
+$EndComp
+$Comp
+L GND #PWR?
+U 1 1 58AB73F7
+P 10200 1000
+F 0 "#PWR?" H 10200 750 50  0001 C CNN
+F 1 "GND" H 10200 850 50  0001 C CNN
+F 2 "" H 10200 1000 50  0000 C CNN
+F 3 "" H 10200 1000 50  0000 C CNN
+	1    10200 1000
+	-1   0    0    1
+$EndComp
+$Comp
+L VCC #PWR?
+U 1 1 58AB76FB
+P 10200 1500
+F 0 "#PWR?" H 10200 1350 50  0001 C CNN
+F 1 "VCC" H 10200 1650 50  0000 C CNN
+F 2 "" H 10200 1500 50  0000 C CNN
+F 3 "" H 10200 1500 50  0000 C CNN
+	1    10200 1500
+	-1   0    0    1
+$EndComp
+Wire Wire Line
+	10000 1100 10200 1100
+Wire Wire Line
+	10200 1100 10200 1000
+Wire Wire Line
+	10000 1200 10200 1200
+Wire Wire Line
+	10200 1200 10200 1500
 $EndSCHEMATC
